File: Flightpad.kicad_sch (KiCad schematic)
At the start: 0 parts

Commit message: Add files via upload
Parts:
- added SW1, SW2, SW3, SW4: SW_Push, Button_Switch_Keyboard:SW_Cherry_MX_1.00u_PCB, symbol Switch:SW_Push
- added SW5: RotaryEncoder_Switch, Rotary_Encoder:RotaryEncoder_Alps_EC11E-Switch_Vertical_H20mm, symbol Device:RotaryEncoder_Switch
- added U1: MOUDLE-SEEEDUINO-XIAO, footprint:XIAO-Generic-Hybrid-14P-2.54-21X17.8MM, symbol XIAO_RP2040:MOUDLE-SEEEDUINO-XIAO
Connections:
- new net: SW1.1, SW2.1, SW3.1, SW4.1, SW5.C, SW5.S2, U1.13 (GND)
- new net: SW4.2, U1.4 (PA11_A3_D3)
- new net: SW2.2, U1.2 (PA4_A1_D1)
- new net: SW3.2, U1.3 (PA10_A2_D2)
- new net: SW1.2, U1.1 (PA02_A0_D0)
- new net: SW5.A, U1.10 (PA5_A9_D9_MISO)
- new net: SW5.S1, U1.11 (PA6_A10_D10_MOSI)
- new net: SW5.B, U1.9 (PA7_A8_D8_SCK)
